Commit message: Update working UR5e sim with fixed mesh paths and launch config

File: archive/ur5e.urdf.xacro (robot description, xacro)
@@ -4,5 +4,5 @@
 <!-- |    EDITING THIS FILE BY HAND IS NOT RECOMMENDED                                 | -->
 <!-- =================================================================================== -->
-<robot name="ur5e">
+<robot xmlns:xacro="http://www.ros.org/wiki/xacro" name="ur5e">
   <!--
     Base UR robot series xacro macro.
@@ -281,3 +281,10 @@
     <child link="tool0"/>
   </joint>
+  <!-- Attach Robotiq 2F-85 Gripper -->
+  <xacro:arg name="use_fake_hardware" default="true" />
+  <xacro:arg name="com_port" default="/dev/ttyUSB0" />
+  <xacro:include filename="$(find robotiq_description)/urdf/robotiq_2f_85_macro.urdf.xacro" />
+  <xacro:robotiq_gripper name="RobotiqGripperHardwareInterface" prefix="" parent="tool0" use_fake_hardware="$(arg use_fake_hardware)" com_port="$(arg com_port)">
+      <origin xyz="0 0 0" rpy="0 0 0" />
+  </xacro:robotiq_gripper>
 </robot>
