Commit message: Removed archive folder and updated package dependencies

File: urdf/inc/ur_common.xacro (robot description, xacro)
@@ -35,5 +35,5 @@
     </xacro:if>
     <xacro:unless value="${force_abs_paths}">
-      <xacro:property name="mesh" value="model://ur5e/${visual_params['mesh']['path']}" scope="parent"/>
+      <xacro:property name="mesh" value="model://ur5e_vla/${visual_params['mesh']['path']}" scope="parent"/>
     </xacro:unless>
   </xacro:macro>

Commit message: Simulation launch method update

File: urdf/inc/ur_common.xacro (robot description, xacro)
@@ -35,5 +35,5 @@
     </xacro:if>
     <xacro:unless value="${force_abs_paths}">
-      <xacro:property name="mesh" value="model://ur5e_vla/${visual_params['mesh']['path']}" scope="parent"/>
+      <xacro:property name="mesh" value="package://ur5e_vla/${visual_params['mesh']['path']}" scope="parent"/>
     </xacro:unless>
   </xacro:macro>

File: urdf/ur5e/OLDur5e.urdf (robot description, URDF)
Before this commit: robot ur5e, 13 links, 12 joints
Links:
- link base_link_inertia: geometry collision mesh filename=model://ur5e_vla/ur5e/collision/base.stl; visual mesh filename=model://ur5e_vla/ur5e/visual/base.dae
- link forearm_link: geometry collision mesh filename=model://ur5e_vla/ur5e/collision/forearm.stl; visual mesh filename=model://ur5e_vla/ur5e/visual/forearm.dae
- link shoulder_link: geometry collision mesh filename=model://ur5e_vla/ur5e/collision/shoulder.stl; visual mesh filename=model://ur5e_vla/ur5e/visual/shoulder.dae
- link upper_arm_link: geometry collision mesh filename=model://ur5e_vla/ur5e/collision/upperarm.stl; visual mesh filename=model://ur5e_vla/ur5e/visual/upperarm.dae
- link wrist_1_link: geometry collision mesh filename=model://ur5e_vla/ur5e/collision/wrist1.stl; visual mesh filename=model://ur5e_vla/ur5e/visual/wrist1.dae
- link wrist_2_link: geometry collision mesh filename=model://ur5e_vla/ur5e/collision/wrist2.stl; visual mesh filename=model://ur5e_vla/ur5e/visual/wrist2.dae
- link wrist_3_link: geometry collision mesh filename=model://ur5e_vla/ur5e/collision/wrist3.stl; visual mesh filename=model://ur5e_vla/ur5e/visual/wrist3.dae
